Commit message: wip

File: kurt_description/robots/kurt360.urdf.xacro (robot description, xacro)
@@ -1,8 +1,8 @@
 <?xml version="1.0"?>
 <robot
-  xmlns:xacro="http://ros.org/wiki/xacro"
-  name="kurt360">
+  xmlns:xacro="http://ros.org/wiki/xacro" name="kurt360">
   <xacro:property name="top_y_offset" value="0.009" />
-  <xacro:property name="base_z_offset" value="0.03" /> <!-- distance from base_link to top of cover surface -->
+  <!-- distance from base_link to top of cover surface -->
+  <xacro:property name="base_z_offset" value="0.03" />
   <xacro:include filename="$(find kurt_base)/urdf/kurt_outdoor.urdf.xacro" />
   <xacro:include filename="$(find kurt_description)/tops/kurt360_top.urdf.xacro" />

File: kurt_description/tops/kurt360_top.urdf.xacro (robot description, xacro)
@@ -1,5 +1,4 @@
 <?xml version="1.0"?>
-<robot
-  xmlns:xacro="http://ros.org/wiki/xacro">
+<robot xmlns:xacro="http://ros.org/wiki/xacro">
   <xacro:include filename="$(find uos_common_urdf)/common.xacro" />
   <xacro:include filename="$(find kurt_base)/urdf/rotunit.urdf.xacro" />
